File: Keyboard.sch (KiCad schematic (older format))
At the start: 109 parts, among them J1 Conn_01x05, J2 Conn_01x08, Q1 BC557, Q2 BC557, Q3 BC557, Q4 BC557, Q5 BC557, Q6 BC557, Q7 BC557, Q8 BC557, SW1 KEY_1, SW10 KEY_0, SW11 KEY_Q, SW12 KEY_W, SW13 KEY_E, SW14 KEY_R, SW15 KEY_T, SW16 KEY_Y, SW17 KEY_U, SW18 KEY_I, SW19 KEY_O, SW2 KEY_2, SW20 KEY_P, SW21 KEY_A, SW22 KEY_S, SW23 KEY_D, SW24 KEY_F, SW25 KEY_G, SW26 KEY_H, SW27 KEY_J, SW28 KEY_K, SW29 KEY_L, SW3 KEY_3, SW30 KEY_ENTER, SW31 KEY_SHIFT, SW32 KEY_Z, SW33 KEY_X, SW34 KEY_C, SW35 KEY_V, SW36 KEY_B, SW37 KEY_N, SW38 KEY_M, SW39 KEY_SYMB, SW4 KEY_4, SW40 KEY_SPACE, SW41 KEY_DOT, SW42 KEY_BREAK, SW43 KEY_COLON, SW44 KEY_COMA, SW45 KEY_DEL, SW46 KEY_SEMICOLON, SW47 KEY_EDIT, SW48 KEY_EQUAL, SW49 KEY_ASTERIC, SW5 KEY_5, SW50 KEY_C_RIGHT, SW51 KEY_C_UP, SW52 KEY_C_DOWN, SW53 KEY_ C_LEFT, SW54 KEY_ EXTRA, SW55 KEY_ GRAF, SW56 KEY_ CAPS_LOCK, SW6 KEY_6, SW7 KEY_7, SW8 KEY_8, SW9 KEY_9, U25 4066, U26 4066

Commit message: add plus 3 disk interface
Parts:
- U25, U26: symbol Logic_CMOS_4000:4066 -> All-Spectrums-rescue:4066-Logic_CMOS_4000
Changed lines of the file:
@@
 $Descr A3 16535 11693
 encoding utf-8
-Sheet 2 16
+Sheet 2 17
 Title ""
 Date ""
@@
 $EndComp
 $Comp
-L Logic_CMOS_4000:4066 U25
+L All-Spectrums-rescue:4066-Logic_CMOS_4000 U25
 U 1 1 5B205FA6
 P 12550 1600
@@
 $EndComp
 $Comp
-L Logic_CMOS_4000:4066 U25
+L All-Spectrums-rescue:4066-Logic_CMOS_4000 U25
 U 2 1 5B20621A
 P 12950 2000
@@
 $EndComp
 $Comp
-L Logic_CMOS_4000:4066 U25
+L All-Spectrums-rescue:4066-Logic_CMOS_4000 U25
 U 3 1 5B2071E6
 P 13350 2400
@@
 $EndComp
 $Comp
-L Logic_CMOS_4000:4066 U25
+L All-Spectrums-rescue:4066-Logic_CMOS_4000 U25
 U 4 1 5B207C80
 P 13750 2800
@@
 	9450 1600 9150 1600
 $Comp
-L Logic_CMOS_4000:4066 U26
+L All-Spectrums-rescue:4066-Logic_CMOS_4000 U26
 U 1 1 5B4F643D
 P 12550 4200
@@
 	12550 4500 13950 4500
 $Comp
-L Logic_CMOS_4000:4066 U26
+L All-Spectrums-rescue:4066-Logic_CMOS_4000 U26
 U 2 1 5B598A3F
 P 12900 5150
@@
 8
 $Comp
-L Logic_CMOS_4000:4066 U26
+L All-Spectrums-rescue:4066-Logic_CMOS_4000 U26
 U 3 1 5B9BAA80
 P 13350 6000
@@
 $EndComp
 $Comp
-L Logic_CMOS_4000:4066 U26
+L All-Spectrums-rescue:4066-Logic_CMOS_4000 U26
 U 4 1 5B9BC4D6
 P 13700 6900
@@
 	12050 6300 12050 6500
 $Comp
-L Logic_CMOS_4000:4066 U25
+L All-Spectrums-rescue:4066-Logic_CMOS_4000 U25
 U 5 1 5BA07275
 P 13650 7900
@@
 $EndComp
 $Comp
-L Logic_CMOS_4000:4066 U26
+L All-Spectrums-rescue:4066-Logic_CMOS_4000 U26
 U 5 1 5BA24F85
 P 14200 7900
