File: PLUSD.sch (KiCad schematic (older format))
At the start: 48 parts, among them J28 Conn_02x17_Odd_Even, J29 Conn_02x13_Odd_Even, SW57 SW_DIP_x02, SW58 SW_DPST_x2, U22 WD1772, U27 AT28C256, U28 74LS00, U29 74LS126, U3 74LS06, U30 74LS175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

Commit message: add plus 3 disk interface
Parts:
- U28: symbol Logic_74xx:74LS00 -> All-Spectrums-rescue:74LS00-Logic_74xx
- U29: symbol Logic_74xx:74LS126 -> All-Spectrums-rescue:74LS126-Logic_74xx
- U3: symbol Logic_74xx:74LS06 -> All-Spectrums-rescue:74LS06-Logic_74xx
- U30: symbol Logic_74xx:74LS175 -> All-Spectrums-rescue:74LS175-Logic_74xx
- U33: symbol Logic_74xx:74LS374 -> All-Spectrums-rescue:74LS374-Logic_74xx
- U34: symbol Logic_74xx:74LS27 -> All-Spectrums-rescue:74LS27-Logic_74xx
Changed lines of the file:
@@
 $Descr A3 16535 11693
 encoding utf-8
-Sheet 14 16
+Sheet 14 17
 Title ""
 Date ""
@@
 $EndComp
 $Comp
-L Logic_74xx:74LS06 U3
+L All-Spectrums-rescue:74LS06-Logic_74xx U3
 U 1 1 5B1B8575
 P 9500 2050
@@
 $EndComp
 $Comp
-L Logic_74xx:74LS06 U3
+L All-Spectrums-rescue:74LS06-Logic_74xx U3
 U 2 1 5B1B85E5
 P 9900 1300
@@
 $EndComp
 $Comp
-L Logic_74xx:74LS06 U3
+L All-Spectrums-rescue:74LS06-Logic_74xx U3
 U 3 1 5B1B8669
 P 9900 1800
@@
 $EndComp
 $Comp
-L Logic_74xx:74LS06 U3
+L All-Spectrums-rescue:74LS06-Logic_74xx U3
 U 6 1 5B1B86AF
 P 9900 2300
@@
 	10650 1300 10200 1300
 $Comp
-L Logic_74xx:74LS06 U3
+L All-Spectrums-rescue:74LS06-Logic_74xx U3
 U 5 1 5B1B862F
 P 9500 1550
@@
 	4650 5650 4750 5650
 $Comp
-L Logic_74xx:74LS00 U28
+L All-Spectrums-rescue:74LS00-Logic_74xx U28
 U 1 1 5B437CE9
 P 8050 3500
@@
 $EndComp
 $Comp
-L Logic_74xx:74LS00 U28
+L All-Spectrums-rescue:74LS00-Logic_74xx U28
 U 2 1 5B437D95
 P 9350 3500
@@
 	6400 3000 6550 3000
 $Comp
-L Logic_74xx:74LS126 U29
+L All-Spectrums-rescue:74LS126-Logic_74xx U29
 U 4 1 5B562568
 P 10000 4250
@@
 $EndComp
 $Comp
-L Logic_74xx:74LS126 U29
+L All-Spectrums-rescue:74LS126-Logic_74xx U29
 U 3 1 5B56D6DE
 P 10250 4650
@@
 $EndComp
 $Comp
-L Logic_74xx:74LS126 U29
+L All-Spectrums-rescue:74LS126-Logic_74xx U29
 U 1 1 5B56D732
 P 10000 5100
@@
 $EndComp
 $Comp
-L Logic_74xx:74LS126 U29
+L All-Spectrums-rescue:74LS126-Logic_74xx U29
 U 5 1 5B5F7599
 P 10050 10400
@@
 $EndComp
 $Comp
-L Logic_74xx:74LS00 U28
+L All-Spectrums-rescue:74LS00-Logic_74xx U28
 U 5 1 5B5F76E6
 P 9600 10400
@@
 $EndComp
 $Comp
-L Logic_74xx:74LS06 U3
+L All-Spectrums-rescue:74LS06-Logic_74xx U3
 U 7 1 5B5F7893
 P 9150 10400
@@
 	2200 10600 2200 10500
 $Comp
-L Logic_74xx:74LS175 U30
+L All-Spectrums-rescue:74LS175-Logic_74xx U30
 U 1 1 5B683FBF
 P 7050 4550
@@
 	8400 2700 11200 2700
 $Comp
-L Logic_74xx:74LS06 U3
+L All-Spectrums-rescue:74LS06-Logic_74xx U3
 U 4 1 5BA454CD
 P 8200 5350
@@
 $EndComp
 $Comp
-L Logic_74xx:74LS374 U33
+L All-Spectrums-rescue:74LS374-Logic_74xx U33
 U 1 1 5B1D5091
 P 9150 7150
@@
 	9700 6250 10750 6250
 $Comp
-L Logic_74xx:74LS126 U29
+L All-Spectrums-rescue:74LS126-Logic_74xx U29
 U 2 1 5B5A0A20
 P 9800 8600
@@
 Connection ~ 1300 7850
 $Comp
-L Logic_74xx:74LS27 U34
+L All-Spectrums-rescue:74LS27-Logic_74xx U34
 U 2 1 5C10F84E
 P 2200 7850
@@
 $EndComp
 $Comp
-L Logic_74xx:74LS00 U28
+L All-Spectrums-rescue:74LS00-Logic_74xx U28
 U 4 1 5C13DCAC
 P 2950 8150
@@
 $EndComp
 $Comp
-L Logic_74xx:74LS27 U34
+L All-Spectrums-rescue:74LS27-Logic_74xx U34
 U 4 1 5C13DF1E
 P 10500 10400
@@
 Connection ~ 10500 9900
 $Comp
-L Logic_74xx:74LS27 U34
+L All-Spectrums-rescue:74LS27-Logic_74xx U34
 U 1 1 5C16DA38
 P 3900 8050
@@
 $EndComp
 $Comp
-L Logic_74xx:74LS27 U34
+L All-Spectrums-rescue:74LS27-Logic_74xx U34
 U 3 1 5C16DB22
 P 3900 8600
@@
 $EndComp
 $Comp
-L Logic_74xx:74LS00 U28
+L All-Spectrums-rescue:74LS00-Logic_74xx U28
 U 3 1 5C16E034
 P 9300 9000
