File: joystick.sch (KiCad schematic (older format))
At the start: 7 parts, among them U19 GAL22V10

Commit message: add plus 3 disk interface
Parts:
- J_ATARI1, J_ATARI2, J_KEMPSTON_ATARI1, J_SJS1, J_SJS2: symbol Connector_Specialized:DB9_Male -> All-Spectrums-rescue:DB9_Male-Connector_Specialized
Changed lines of the file:
@@
 $Descr A4 11693 8268
 encoding utf-8
-Sheet 10 16
+Sheet 10 17
 Title ""
 Date ""
@@
 $EndDescr
 $Comp
-L Connector_Specialized:DB9_Male J_SJS2
+L All-Spectrums-rescue:DB9_Male-Connector_Specialized J_SJS2
 U 1 1 5B860AA3
 P 5900 3200
@@
 $EndComp
 $Comp
-L Connector_Specialized:DB9_Male J_SJS1
+L All-Spectrums-rescue:DB9_Male-Connector_Specialized J_SJS1
 U 1 1 5B860B89
 P 5900 1700
@@
 $EndComp
 $Comp
-L Connector_Specialized:DB9_Male J_ATARI1
+L All-Spectrums-rescue:DB9_Male-Connector_Specialized J_ATARI1
 U 1 1 5B860BEF
 P 8350 1700
@@
 $EndComp
 $Comp
-L Connector_Specialized:DB9_Male J_ATARI2
+L All-Spectrums-rescue:DB9_Male-Connector_Specialized J_ATARI2
 U 1 1 5B860C15
 P 8350 3150
@@
 $EndComp
 $Comp
-L Connector_Specialized:DB9_Male J_KEMPSTON_ATARI1
+L All-Spectrums-rescue:DB9_Male-Connector_Specialized J_KEMPSTON_ATARI1
 U 1 1 5B860C77
 P 8350 5100
