File: power.sch (KiCad schematic (older format))
At the start: 20 parts, among them J4 Jack-DC, U10 AP1117-33, U11 LM2596S-5, U12 74HC04, U2 L7805, U6 74HC04, Y4 14.000Mhz

Commit message: add plus 3 disk interface
Parts:
- J4: symbol Connector_Specialized:Jack-DC -> All-Spectrums-rescue:Jack-DC-Connector_Specialized
- U12, U6: symbol Logic_74xx:74HC04 -> All-Spectrums-rescue:74HC04-Logic_74xx
Changed lines of the file:
@@
 $Descr A4 11693 8268
 encoding utf-8
-Sheet 4 16
+Sheet 4 17
 Title ""
 Date ""
@@
 $EndDescr
 $Comp
-L Connector_Specialized:Jack-DC J4
+L All-Spectrums-rescue:Jack-DC-Connector_Specialized J4
 U 1 1 5B2FBCC4
 P 1350 1600
@@
 	5750 1900 5750 1950
 $Comp
-L Logic_74xx:74HC04 U?
+L All-Spectrums-rescue:74HC04-Logic_74xx U?
 U 1 1 5B6F02A6
 P 1850 6150
@@
 $EndComp
 $Comp
-L Logic_74xx:74HC04 U?
+L All-Spectrums-rescue:74HC04-Logic_74xx U?
 U 2 1 5B6F02AD
 P 2850 6150
@@
 $EndComp
 $Comp
-L Logic_74xx:74HC04 U?
+L All-Spectrums-rescue:74HC04-Logic_74xx U?
 U 3 1 5B6F02B4
 P 3500 6150
@@
 $EndComp
 $Comp
-L Logic_74xx:74HC04 U?
+L All-Spectrums-rescue:74HC04-Logic_74xx U?
 U 7 1 5BA0F3B8
 P 5700 6600
