File: psg.sch (KiCad schematic (older format))
At the start: 47 parts, among them J17 Conn_02x04_Odd_Even, J18 Audio-Jack-3_2Switches, J19 Conn_02x04_Odd_Even, J20 RJ45, J21 DB9_Female, J22 Conn_01x10, J23 RJ45, U13 MAX232, U14 PSG_AY-3-8910, U15 PSG_AY-3-8912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

Commit message: add plus 3 disk interface
Parts:
- J18: symbol Connector_Specialized:Audio-Jack-3_2Switches -> All-Spectrums-rescue:Audio-Jack-3_2Switches-Connector_Specialized
- J20, J23: symbol Connector_Specialized:RJ45 -> All-Spectrums-rescue:RJ45-Connector_Specialized
- J21: symbol Connector_Specialized:DB9_Female -> All-Spectrums-rescue:DB9_Female-Connector_Specialized
- U17: symbol Logic_74xx:74HC00 -> All-Spectrums-rescue:74HC00-Logic_74xx
- U18: symbol Logic_74xx:74HC74 -> All-Spectrums-rescue:74HC74-Logic_74xx
Changed lines of the file:
@@
 $Descr A4 11693 8268
 encoding utf-8
-Sheet 9 16
+Sheet 9 17
 Title ""
 Date ""
@@
 	4450 2100 4450 2150
 $Comp
-L Logic_74xx:74HC74 U18
+L All-Spectrums-rescue:74HC74-Logic_74xx U18
 U 1 1 5B1705C4
 P 2700 6400
@@
 $EndComp
 $Comp
-L Logic_74xx:74HC00 U17
+L All-Spectrums-rescue:74HC00-Logic_74xx U17
 U 2 1 5B170749
 P 1150 6400
@@
 $EndComp
 $Comp
-L Logic_74xx:74HC00 U17
+L All-Spectrums-rescue:74HC00-Logic_74xx U17
 U 4 1 5B17082C
 P 2000 6400
@@
 $EndComp
 $Comp
-L Logic_74xx:74HC00 U17
+L All-Spectrums-rescue:74HC00-Logic_74xx U17
 U 5 1 5B21716E
 P 3950 6900
@@
 $EndComp
 $Comp
-L Logic_74xx:74HC74 U18
+L All-Spectrums-rescue:74HC74-Logic_74xx U18
 U 3 1 5B2171EA
 P 4900 6900
@@
 	9100 2050 9250 2050
 $Comp
-L Connector_Specialized:RJ45 J20
+L All-Spectrums-rescue:RJ45-Connector_Specialized J20
 U 1 1 5B3206FA
 P 10300 2600
@@
 	9100 5000 9250 5000
 $Comp
-L Connector_Specialized:RJ45 J23
+L All-Spectrums-rescue:RJ45-Connector_Specialized J23
 U 1 1 5B3F0B3B
 P 10300 5550
@@
 	8800 5800 8700 5800
 $Comp
-L Connector_Specialized:DB9_Female J21
+L All-Spectrums-rescue:DB9_Female-Connector_Specialized J21
 U 1 1 5B492676
 P 10250 3650
@@
 $EndComp
 $Comp
-L Connector_Specialized:Audio-Jack-3_2Switches J18
+L All-Spectrums-rescue:Audio-Jack-3_2Switches-Connector_Specialized J18
 U 1 1 5B155254
 P 4250 1900
