File: sound.sch (KiCad schematic (older format))
At the start: 30 parts, among them J15 EAR, J16 PLUS3_EAR_MIC, J5 EAR, J6 MIC, J9 Conn_01x03, Q14 BC848, Q9 BC548, U8 TL712

Commit message: add plus 3 disk interface
Parts:
- J15, J16, J5, J6: symbol Connector_Specialized:Audio-Jack-3_2Switches -> All-Spectrums-rescue:Audio-Jack-3_2Switches-Connector_Specialized
Changed lines of the file:
@@
 $Descr A4 11693 8268
 encoding utf-8
-Sheet 5 16
+Sheet 5 17
 Title ""
 Date ""
@@
 $EndDescr
 $Comp
-L Connector_Specialized:Audio-Jack-3_2Switches J5
+L All-Spectrums-rescue:Audio-Jack-3_2Switches-Connector_Specialized J5
 U 1 1 5B306A4F
 P 4800 1600
@@
 $EndComp
 $Comp
-L Connector_Specialized:Audio-Jack-3_2Switches J6
+L All-Spectrums-rescue:Audio-Jack-3_2Switches-Connector_Specialized J6
 U 1 1 5B306B5F
 P 4800 3650
@@
 NoConn ~ 4600 1500
 $Comp
-L Connector_Specialized:Audio-Jack-3_2Switches J16
+L All-Spectrums-rescue:Audio-Jack-3_2Switches-Connector_Specialized J16
 U 1 1 5B593E48
 P 4800 2700
@@
 	4450 2600 4600 2600
 $Comp
-L Connector_Specialized:Audio-Jack-3_2Switches J15
+L All-Spectrums-rescue:Audio-Jack-3_2Switches-Connector_Specialized J15
 U 1 1 5BA60F92
 P 8700 1500
