File: ula_MAX.sch (KiCad schematic (older format))
At the start: 11 parts, among them J10 JTAG, U6 74HC04, U7 EPM7128S_LCC

Commit message: add plus 3 disk interface
Parts:
- U6: symbol Logic_74xx:74HC04 -> All-Spectrums-rescue:74HC04-Logic_74xx
Changed lines of the file:
@@
 $Descr A4 11693 8268
 encoding utf-8
-Sheet 7 16
+Sheet 7 17
 Title ""
 Date ""
@@
 Connection ~ 9350 1100
 $Comp
-L Logic_74xx:74HC04 U6
+L All-Spectrums-rescue:74HC04-Logic_74xx U6
 U 7 1 5B56995C
 P 10900 1350
