File: video.sch (KiCad schematic (older format))
At the start: 55 parts, among them J11 Conn_01x03, J12 Mini-DIN-8, J13 Conn_01x03, J14 Conn_01x03, J7 VIDEO, Q10 BC548, Q11 BC548, Q12 BC548, Q13 BC548, U6 74HC04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

Commit message: add plus 3 disk interface
Parts:
- J12: symbol Connector_Specialized:Mini-DIN-8 -> All-Spectrums-rescue:Mini-DIN-8-Connector_Specialized
- J7: symbol Connector_Specialized:Conn_Coaxial -> All-Spectrums-rescue:Conn_Coaxial-Connector_Specialized
- U6: symbol Logic_74xx:74HC04 -> All-Spectrums-rescue:74HC04-Logic_74xx
Changed lines of the file:
@@
 $Descr A4 11693 8268
 encoding utf-8
-Sheet 8 16
+Sheet 8 17
 Title ""
 Date ""
@@
 $EndDescr
 $Comp
-L Connector_Specialized:Conn_Coaxial J7
+L All-Spectrums-rescue:Conn_Coaxial-Connector_Specialized J7
 U 1 1 5B306826
 P 10700 2200
@@
 bright
 $Comp
-L Logic_74xx:74HC04 U?
+L All-Spectrums-rescue:74HC04-Logic_74xx U?
 U 4 1 5B536EF3
 P 1000 5550
@@
 $EndComp
 $Comp
-L Logic_74xx:74HC04 U?
+L All-Spectrums-rescue:74HC04-Logic_74xx U?
 U 5 1 5B536EFA
 P 2000 5550
@@
 $EndComp
 $Comp
-L Logic_74xx:74HC04 U?
+L All-Spectrums-rescue:74HC04-Logic_74xx U?
 U 6 1 5B536F01
 P 2650 5550
@@
 Connection ~ 9600 2200
 $Comp
-L Connector_Specialized:Mini-DIN-8 J12
+L All-Spectrums-rescue:Mini-DIN-8-Connector_Specialized J12
 U 1 1 5B60CF5D
 P 9050 4400
