File: wilcodisk.sch (KiCad schematic (older format))
At the start: 6 parts, among them J24 WILCO's_FLOPPY_INTERFAZ, J25 IDE_8bits, J26 cartridge_IF2, U23 7410

Commit message: add plus 3 disk interface
Parts:
- U23: symbol Logic_TTL_IEEE:7410 -> All-Spectrums-rescue:7410-Logic_TTL_IEEE
Connections:
- net labels removed: RESET, RW
- wire segments 87 -> 89
- no-connect marks 29 -> 27
Changed lines of the file:
@@
 $Descr A4 11693 8268
 encoding utf-8
-Sheet 12 16
+Sheet 12 17
 Title ""
 Date ""
@@
 A15
 Text GLabel 2550 2100 2    50   Input ~ 0
-RW
+WR
 Text GLabel 1700 2100 0    50   Input ~ 0
 RD
 Text GLabel 2550 2200 2    50   Input ~ 0
 IOREQ
-Text GLabel 1700 2200 0    50   Input ~ 0
-RESET
+Text GLabel 1400 2200 0    50   Input ~ 0
+~RESET
 $Comp
 L power:+5V #PWR0207
@@
 	2450 2200 2550 2200
 Wire Wire Line
-	1700 2200 1950 2200
+	1400 2200 1950 2200
 Wire Wire Line
 	1700 2100 1950 2100
@@
 NoConn ~ 1950 1500
 NoConn ~ 1950 1600
-NoConn ~ 1950 1200
-NoConn ~ 1950 1700
 Text GLabel 2700 1200 2    50   Input ~ 0
 D0
@@
 $EndComp
 $Comp
-L Logic_TTL_IEEE:7410 U23
+L All-Spectrums-rescue:7410-Logic_TTL_IEEE U23
 U 1 1 5B1A7486
 P 2300 5550
@@
 $EndComp
 $Comp
-L Logic_TTL_IEEE:7410 U23
+L All-Spectrums-rescue:7410-Logic_TTL_IEEE U23
 U 3 1 5B1A754C
 P 2300 6200
@@
 $EndComp
 $Comp
-L Logic_TTL_IEEE:7410 U23
+L All-Spectrums-rescue:7410-Logic_TTL_IEEE U23
 U 2 1 5B1A75C7
 P 3500 5850
@@
 	1    0    0    -1
 $EndComp
+Text GLabel 1700 1700 0    50   Input ~ 0
+A12
+Text GLabel 1700 1200 0    50   Input ~ 0
+D3
+Wire Wire Line
+	1700 1200 1950 1200
+Wire Wire Line
+	1700 1700 1950 1700
 $EndSCHEMATC
